Commit message: simple_terrain, updated urdf

File: urdf/turtlebot3_waffle.urdf (robot description, URDF)
Before this commit: robot turtlebot3_waffle, 13 links, 12 joints
Links:
- removed link camera_depth_frame
- removed link camera_depth_optical_frame
- removed link camera_link
- removed link camera_rgb_frame
- removed link camera_rgb_optical_frame
Joints:
- removed joint camera_depth_joint
- removed joint camera_depth_optical_joint
- removed joint camera_joint
- removed joint camera_rgb_joint
- removed joint camera_rgb_optical_joint
- joint scan_joint: origin xyz=-0.064 0 0.122 rpy=0 0 0 -> xyz=0 0 0.121 rpy=0 0 0

Commit message: terrain map

File: urdf/turtlebot3_waffle.urdf (robot description, URDF)
Before this commit: robot turtlebot3_waffle, 8 links, 7 joints
Links:
- added link base_lidar, mass 0.114; collision cylinder length=0.0315 radius=0.055; visual mesh filename=package://turtlebot3_gazebo/models/turtlebot3_common/meshes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 scale=0.001 0.001 0.001
Joints:
- added joint lidar_joint: type fixed, parent base_link, child base_lidar, origin xyz=0 0 0.121 rpy=0 0 0

Commit message: nav2 waypoint follower

File: urdf/turtlebot3_waffle.urdf (robot description, URDF)
Before this commit: robot turtlebot3_waffle, 9 links, 8 joints
Links:
- link base_lidar: geometry visual mesh filename=package://turtlebot3_gazebo/models/turtlebot3_common/meshes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 scale=0.001 0.001 0.001
