Commit message: flat tree terrain

File: urdf/turtlebot3_burger.urdf (robot description, URDF)
Before this commit: robot turtlebot3_burger, 7 links, 6 joints
Links:
- added link base_lidar, mass 0.114; visual mesh filename=package://turtlebot3_gazebo/models/turtlebot3_common/meshes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 scale=0.001 0.001 0.001
Joints:
- added joint lidar_joint: type fixed, parent base_link, child base_lidar, origin xyz=0 0 0.172 rpy=0 0 3.141
- joint scan_joint: origin xyz=-0.032 0 0.172 rpy=0 0 0 -> xyz=0 0 0.172 rpy=0 0 3.141
